File: hardware/Controller v1.0/controller v1.brd (EAGLE design)
At the start: 71.1 x 73.1 mm, 36 parts, among them CON1 1X08-CONN3.5MM, CON2 1X08-CONN3.5MM, CON3 1X08-CONN3.5MM, CON4 1X08-CONN3.5MM, IC1 MC33880PEG, IC2 L293DD, IC3 MC33880PEG

Commit message: Updates to match exactly first working prototype
Parts:
- C1: value 220n -> 100n
- C13: value (none) -> 100n
- R5: value 50m -> 100m
- R6: value 10k -> 5.1k
- R7: value (none) -> 10k
Changed lines of the file:
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@@
 <element name="R3" library="resistor" package="R0805" value="10k" x="68.834" y="23.876"/>
 <element name="SL2" library="adafruit" package="1X2-3.5MM" value="1X2-3.5MM" x="83.82" y="40.64" rot="R90"/>
-<element name="C1" library="resistor" package="C0805" value="220n" x="68.834" y="21.209" rot="R180"/>
+<element name="C1" library="resistor" package="C0805" value="100n" x="68.834" y="21.209" rot="R180"/>
 <element name="C2" library="rcl-ez" package="C025-025X050" value="0.1uF" x="69.088" y="30.099" rot="R90"/>
 <element name="C3" library="rcl-ez" package="C025-025X050" value="0.1uF" x="51.308" y="27.559" rot="R270"/>
@@
 <element name="R4" library="rcl-ez" package="M0805" value="1.0K" x="80.772" y="47.244"/>
 <element name="PWR" library="minimidi" package="LED3MM" value="" x="81.28" y="51.308" rot="R90"/>
-<element name="R5" library="resistor" package="M1206" value="50m" x="51.054" y="19.939"/>
-<element name="R6" library="resistor" package="R0603" value="10k" x="63.754" y="16.891" rot="R180"/>
-<element name="R7" library="resistor" package="R0603" value="" x="63.754" y="14.605" rot="R180"/>
-<element name="C13" library="resistor" package="C0805K" value="" x="67.818" y="16.129" rot="R90"/>
+<element name="R5" library="resistor" package="M1206" value="100m" x="51.054" y="19.939"/>
+<element name="R6" library="resistor" package="R0603" value="5.1k" x="63.754" y="16.891" rot="R180"/>
+<element name="R7" library="resistor" package="R0603" value="10k" x="63.754" y="14.605" rot="R180"/>
+<element name="C13" library="resistor" package="C0805K" value="100n" x="67.818" y="16.129" rot="R90"/>
 <element name="U$3" library="aerodynes" package="SOT23-1TOP" value="ZXCT1009-F" x="59.436" y="16.891" rot="R270"/>
 <element name="JP1" library="jumper" package="JP1" value="" x="46.99" y="16.256"/>

Commit message: Another slight update for component values
Parts:
- C6, C9: value 10uF 20V -> 100uF 25V
- C7: value 100uF/16V -> 330uF/25V
Changed lines of the file:
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@@
 <element name="U$1" library="aerodynes" package="ARDUINO-NOCUT" value="ARDUINO" x="30.48" y="45.466"/>
 <element name="C4" library="adafruit" package="E2,5-5" value="100uF/6V" x="64.516" y="36.068" rot="R90"/>
-<element name="C7" library="rcl-ez" package="E2,5-6" value="100uF/16V" x="74.93" y="40.64" rot="R270"/>
+<element name="C7" library="rcl-ez" package="E2,5-6" value="330uF/25V" x="74.93" y="40.64" rot="R270"/>
 <element name="R1" library="resistor" package="R0805" value="10k" x="73.152" y="24.638" rot="R90"/>
 <element name="R2" library="resistor" package="R0805" value="10k" x="73.152" y="19.939" rot="R270"/>
@@
 <element name="IC1" library="aerodynes" package="SO28W" value="MC33880PEG" x="40.64" y="39.37" rot="R270"/>
 <element name="IC3" library="aerodynes" package="SO28W" value="MC33880PEG" x="36.83" y="20.32"/>
-<element name="C6" library="rcl" package="E2,5-6E" value="10uF 20V" x="46.482" y="54.864"/>
+<element name="C6" library="rcl" package="E2,5-6E" value="100uF 25V" x="46.482" y="54.864"/>
 <element name="C8" library="rcl-ez" package="C025-025X050" value="0.1uF 6V" x="21.082" y="26.924" rot="R180"/>
-<element name="C9" library="rcl" package="E2,5-6E" value="10uF 20V" x="21.082" y="21.59" rot="R180"/>
+<element name="C9" library="rcl" package="E2,5-6E" value="100uF 25V" x="21.082" y="21.59" rot="R180"/>
 <element name="C10" library="rcl-ez" package="C025-025X050" value="0.1uF 6V" x="39.878" y="54.61"/>
 <element name="C11" library="rcl-ez" package="C0805K" value="1pF 6V" x="38.1" y="31.75"/>

Commit message: Add support for current sensor.
All values output by the controller are now in real units (mV for BEMF
and mA for current). Web app graphs current value. Better graphs (no
gaps when sending turnout commands).
Parts:
- C13: value 100n -> 10n
- R7: value 10k -> 33k
Changed lines of the file:
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@@
 <element name="R5" library="resistor" package="M1206" value="100m" x="51.054" y="19.939"/>
 <element name="R6" library="resistor" package="R0603" value="5.1k" x="63.754" y="16.891" rot="R180"/>
-<element name="R7" library="resistor" package="R0603" value="10k" x="63.754" y="14.605" rot="R180"/>
-<element name="C13" library="resistor" package="C0805K" value="100n" x="67.818" y="16.129" rot="R90"/>
+<element name="R7" library="resistor" package="R0603" value="33k" x="63.754" y="14.605" rot="R180"/>
+<element name="C13" library="resistor" package="C0805K" value="10n" x="67.818" y="16.129" rot="R90"/>
 <element name="U$3" library="aerodynes" package="SOT23-1TOP" value="ZXCT1009-F" x="59.436" y="16.891" rot="R270"/>
 <element name="JP1" library="jumper" package="JP1" value="" x="46.99" y="16.256"/>
